Commit message: updated urdf with inertia and collision

File: sbrobot_desc/urdf/sbrobot.urdf (robot description, URDF)
Before this commit: robot jetPR, 3 links, 2 joints
Links:
- link base_link: mass None -> 5.0; geometry collision box size=.2 .3 .5; visual box size=.2 .3 .5
- link left_wheel: mass None -> .5; geometry collision cylinder length=0.05 radius=0.1; visual cylinder length=0.05 radius=0.1
- link right_wheel: mass None -> 0.5; geometry collision cylinder length=0.05 radius=0.1; visual cylinder length=0.05 radius=0.1
Joints:
- joint left_wheel_hinge: limit (none) -> effort=1.5 velocity=100
- joint right_wheel_hinge: limit (none) -> effort=1.5 velocity=100

Commit message: added imu to urdf

File: sbrobot_desc/urdf/sbrobot.urdf (robot description, URDF)
Before this commit: robot jetPR, 3 links, 2 joints
Links:
- added link base_footprint
- added link head, mass 0.1; collision box size=.1 .1 .1; visual box size=.1 .1 .1
Joints:
- added joint dummy_joint: type fixed, parent base_footprint, child base_link, origin xyz=0 0.0 0 rpy=0 0 0
- added joint head_joint: type fixed, parent base_link, child head, origin xyz=0 0.0 0.55 rpy=0 0 0

Commit message: changed limits

File: sbrobot_desc/urdf/sbrobot.urdf (robot description, URDF)
Before this commit: robot jetPR, 5 links, 4 joints
Joints:
- joint left_wheel_hinge: limit effort=1.5 velocity=100 -> effort=1.5 velocity=1000000
- joint right_wheel_hinge: limit effort=1.5 velocity=100 -> effort=1.5 velocity=1000000

Commit message: updated max speeds

File: sbrobot_desc/urdf/sbrobot.urdf (robot description, URDF)
Before this commit: robot jetPR, 5 links, 4 joints
Joints:
- joint left_wheel_hinge: limit effort=1.5 velocity=1000000 -> effort=1.5 velocity=1000
- joint right_wheel_hinge: limit effort=1.5 velocity=1000000 -> effort=1.5 velocity=1000
